Commit message: initial commit for hacky success with Khepri and jackal_velodyne

File: jackal_description/urdf/accessories.urdf.xacro (robot description, xacro)
@@ -17,13 +17,23 @@
     <xacro:if value="$(optenv JACKAL_LASER_HOKUYO 0)">
       <xacro:include filename="$(find jackal_description)/urdf/accessories/hokuyo_ust10.urdf.xacro" />
-      <xacro:hokuyo_ust10_mount prefix="$(optenv JACKAL_LASER_MOUNT front)"
-                          parent_link="$(optenv JACKAL_LASER_MOUNT front)_mount"
+      <hokuyo_ust10_mount prefix="$(optenv JACKAL_LASER_MOUNT front)"
                           topic="$(optenv JACKAL_LASER_TOPIC front/scan)" />
+      <joint name="$(optenv JACKAL_LASER_MOUNT front)_laser_mount_joint" type="fixed">
+        <origin xyz="$(optenv JACKAL_LASER_OFFSET 0.11 0 0)"
+                rpy="$(optenv JACKAL_LASER_RPY 0 0 0)" />
+        <parent link="$(optenv JACKAL_LASER_MOUNT front)_mount" />
+        <child link="$(optenv JACKAL_LASER_MOUNT front)_laser_mount" />
+      </joint>
     </xacro:if>
     <xacro:unless value="$(optenv JACKAL_LASER_HOKUYO 0)">
       <xacro:include filename="$(find jackal_description)/urdf/accessories/sick_lms1xx_mount.urdf.xacro" />
-      <xacro:sick_lms1xx_mount prefix="$(optenv JACKAL_LASER_MOUNT front)"
-                         parent_link="$(optenv JACKAL_LASER_MOUNT front)_mount"
+      <sick_lms1xx_mount prefix="$(optenv JACKAL_LASER_MOUNT front)"
                          topic="$(optenv JACKAL_LASER_TOPIC front/scan)"/>
+      <joint name="$(optenv JACKAL_LASER_MOUNT front)_laser_mount_joint" type="fixed">
+        <origin xyz="$(optenv JACKAL_LASER_OFFSET 0 0 0)"
+                rpy="$(optenv JACKAL_LASER_RPY 0 0 0)" />
+        <parent link="$(optenv JACKAL_LASER_MOUNT front)_mount" />
+        <child link="$(optenv JACKAL_LASER_MOUNT front)_laser_mount" />
+      </joint>
     </xacro:unless>
   </xacro:if>
@@ -31,7 +41,7 @@
   <xacro:if value="$(optenv JACKAL_NAVSAT 0)">
     <xacro:include filename="$(find jackal_description)/urdf/accessories/novatel_smart6.urdf.xacro" />
-    <xacro:bridge_plate mount="$(optenv JACKAL_NAVSAT_MOUNT rear)"
+    <bridge_plate mount="$(optenv JACKAL_NAVSAT_MOUNT rear)"
                   height="$(optenv JACKAL_NAVSAT_HEIGHT 0.1)" />
-    <xacro:novatel_smart6 prefix="$(optenv JACKAL_NAVSAT_MOUNT rear)"/>
+    <novatel_smart6 prefix="$(optenv JACKAL_NAVSAT_MOUNT rear)"/>
     <joint name="$(optenv JACKAL_NAVSAT_MOUNT rear)_navsat_joint" type="fixed">
       <origin xyz="0 0 0" rpy="0 0 0" />
@@ -41,9 +51,9 @@
   </xacro:if>
   <!-- Common camera mounts and accessory URDFs. -->
-  <xacro:include filename="$(find jackal_description)/urdf/accessories/camera_mount.urdf.xacro" />
-  <xacro:include filename="$(find pointgrey_camera_description)/urdf/pointgrey_flea3.urdf.xacro" />
+  <!-- <xacro:include filename="$(find jackal_description)/urdf/accessories/camera_mount.urdf.xacro" /> -->
+  <!-- <xacro:include filename="$(find pointgrey_camera_description)/urdf/pointgrey_flea3.urdf.xacro" /> -->
   <!-- If enabled, generate the flea3 camera payload with a tilt of 30 degrees. -->
-  <xacro:if value="$(optenv JACKAL_FLEA3 0)">
-    <xacro:camera_mount prefix="$(optenv JACKAL_FLEA3_MOUNT front)"
+  <!-- <xacro:if value="$(optenv JACKAL_FLEA3 0)">
+    <camera_mount prefix="$(optenv JACKAL_FLEA3_MOUNT front)"
                        tilt="$(optenv JACKAL_FLEA3_TILT 0.5236)"/>
     <joint name="$(optenv JACKAL_FLEA3_MOUNT front)_camera_mount_joint" type="fixed">
@@ -53,5 +63,5 @@
       <child link="$(optenv JACKAL_FLEA3_MOUNT front)_camera_mount" />
     </joint>
-    <xacro:pointgrey_flea3 frame="$(optenv JACKAL_FLEA3_MOUNT front)_camera" name="$(optenv JACKAL_FLEA3_NAME front)"
+    <pointgrey_flea3 frame="$(optenv JACKAL_FLEA3_MOUNT front)_camera" name="$(optenv JACKAL_FLEA3_NAME front)"
       camera_x="0.0754" camera_y="0.029" camera_z="0.029"
       camera_mass="0.085" hfov="1.0471975512" fps="60" width="640" height="512"/>
@@ -61,10 +71,10 @@
       <child link="$(optenv JACKAL_FLEA3_MOUNT front)_camera" />
     </joint>
-  </xacro:if>
-  <xacro:include filename="$(find jackal_description)/urdf/accessories/stereo_camera_mount.urdf.xacro" />
+  </xacro:if> -->
+  <!-- <xacro:include filename="$(find jackal_description)/urdf/accessories/stereo_camera_mount.urdf.xacro" /> -->
   <!-- If enabled, generates a pair of flea3 cameras for stereo vision with a tilt of 30 degrees. -->
   <!-- Disabled temporarily due to metapackage issue. -->
-  <xacro:if value="$(optenv JACKAL_STEREO_FLEA3 0)">
-    <xacro:stereo_camera_mount prefix="$(optenv JACKAL_FLEA3_MOUNT front)"
+  <!-- <xacro:if value="$(optenv JACKAL_STEREO_FLEA3 0)">
+    <stereo_camera_mount prefix="$(optenv JACKAL_FLEA3_MOUNT front)"
                        tilt="$(optenv JACKAL_FLEA3_TILT 0.5236)"/>
     <joint name="$(optenv JACKAL_FLEA3_MOUNT front)_stereo_camera_mount_joint" type="fixed">
@@ -74,5 +84,5 @@
       <child link="$(optenv JACKAL_FLEA3_MOUNT front)_stereo_camera_mount" />
     </joint>
-    <xacro:pointgrey_flea3 frame="$(optenv JACKAL_FLEA3_MOUNT front)_left_camera" name="$(optenv JACKAL_FLEA3_LEFT_NAME front/left)"
+    <pointgrey_flea3 frame="$(optenv JACKAL_FLEA3_MOUNT front)_left_camera" name="$(optenv JACKAL_FLEA3_LEFT_NAME front/left)"
       camera_x="0.0754" camera_y="0.029" camera_z="0.029"
       camera_mass="0.085" hfov="1.0471975512" fps="60" width="640" height="512"/>
@@ -82,5 +92,5 @@
       <child link="$(optenv JACKAL_FLEA3_MOUNT front)_left_camera" />
     </joint>
-    <xacro:pointgrey_flea3 frame="$(optenv JACKAL_FLEA3_MOUNT front)_right_camera" name="$(optenv JACKAL_FLEA3_RIGHT_NAME front/right)"
+    <pointgrey_flea3 frame="$(optenv JACKAL_FLEA3_MOUNT front)_right_camera" name="$(optenv JACKAL_FLEA3_RIGHT_NAME front/right)"
       camera_x="0.0754" camera_y="0.029" camera_z="0.029"
       camera_mass="0.085" hfov="1.0471975512" fps="60" width="640" height="512"/>
@@ -90,11 +100,11 @@
       <child link="$(optenv JACKAL_FLEA3_MOUNT front)_right_camera" />
     </joint>
-  </xacro:if>
+  </xacro:if> -->
   <!-- If enabled, generate the bumblebee2 camera payload with a tilt of 0 degrees. -->
-  <xacro:include filename="$(find pointgrey_camera_description)/urdf/pointgrey_bumblebee2.urdf.xacro" />
+  <!-- <xacro:include filename="$(find pointgrey_camera_description)/urdf/pointgrey_bumblebee2.urdf.xacro" /> -->
   <!-- If enabled, generate the bumblebee2 camera payload with a tilt of 0 degrees. -->
   <!-- Disabled temporarily due to metapackage issue. -->
-  <xacro:if value="$(optenv JACKAL_BB2 0)">
-    <xacro:camera_mount prefix="$(optenv JACKAL_BB2_MOUNT front)"
+  <!-- <xacro:if value="$(optenv JACKAL_BB2 0)">
+    <camera_mount prefix="$(optenv JACKAL_BB2_MOUNT front)"
                         tilt="$(optenv JACKAL_BB2_TILT 0)"/>
     <joint name="$(optenv JACKAL_BB2_MOUNT front)_camera_mount_joint" type="fixed">
@@ -104,5 +114,5 @@
       <child link="$(optenv JACKAL_BB2_MOUNT front)_camera_mount" />
     </joint>
-    <xacro:BB2-08S2C-38 frame="$(optenv JACKAL_BB2_MOUNT front)_camera" name="$(optenv JACKAL_BB2_NAME front)" />
+    <BB2-08S2C-38 frame="$(optenv JACKAL_BB2_MOUNT front)_camera" name="$(optenv JACKAL_BB2_NAME front)" />
     <joint name="$(optenv JACKAL_BB2_MOUNT front)_camera_bracket_joint" type="fixed">
       <origin xyz="0.007 0 0.02450" rpy="0 0 0" />
@@ -110,20 +120,14 @@
       <child link="$(optenv JACKAL_BB2_MOUNT front)_camera" />
     </joint>
-  </xacro:if>
+  </xacro:if> -->
   <xacro:if value="$(optenv JACKAL_FRONT_ACCESSORY_FENDER 0)">
     <xacro:include filename="$(find jackal_description)/urdf/accessories/hokuyo_ust10.urdf.xacro" />
     <xacro:if value="$(optenv JACKAL_FRONT_FENDER_UST10 0)">
-      <xacro:hokuyo_ust10_mount
-        prefix="front"
-        parent_link="front_fender_accessory_link"
-        topic="$(optenv JACKAL_FRONT_LASER_TOPIC front/scan)"/>
+        <hokuyo_ust10 prefix="front_ust10" parent_link="front_fender_accessory_link"/>
     </xacro:if>
   </xacro:if>
   <xacro:if value="$(optenv JACKAL_REAR_ACCESSORY_FENDER 0)">
     <xacro:if value="$(optenv JACKAL_REAR_FENDER_UST10 0)">
-      <xacro:hokuyo_ust10_mount
-        prefix="rear"
-        parent_link="rear_fender_accessory_link"
-        topic="$(optenv JACKAL_REAR_LASER_TOPIC rear/scan)"/>
+        <hokuyo_ust10 prefix="rear_ust10" parent_link="rear_fender_accessory_link"/>
     </xacro:if>
   </xacro:if>

File: jackal_description/urdf/accessories/hokuyo_ust10.urdf.xacro (robot description, xacro)
@@ -1,5 +1,5 @@
 <?xml version="1.0"?>
 <robot xmlns:xacro="http://ros.org/wiki/xacro">
-  <xacro:macro name="hokuyo_ust10_mount" params="prefix topic parent_link">
+  <xacro:macro name="hokuyo_ust10_mount" params="prefix topic">
     <xacro:macro name="hokuyo_ust10" params="frame:=laser topic:=scan sample_size:=720 update_rate:=50
                min_angle:=-2.35619 max_angle:=2.35619 min_range:=0.1 max_range:=30.0 robot_namespace:=/">
@@ -47,11 +47,5 @@
       </gazebo>
     </xacro:macro>
-    <xacro:hokuyo_ust10 frame="${prefix}_laser" topic="${topic}"/>
-    <joint name="${prefix}_laser_mount_joint" type="fixed">
-      <origin xyz="$(optenv JACKAL_LASER_OFFSET 0 0 0)"
-              rpy="$(optenv JACKAL_LASER_RPY 0 0 0)" />
-      <parent link="${parent_link}" />
-      <child link="${prefix}_laser_mount" />
-    </joint>
+    <hokuyo_ust10 frame="${prefix}_laser" topic="${topic}" />
     <link name="${prefix}_laser_mount">
       <visual>
@@ -66,5 +60,5 @@
     <joint name="${prefix}_laser_joint" type="fixed">
       <!-- This offset is from the base of the bracket to the LIDAR's focal point. -->
-      <origin xyz="0 0 0.0474" rpy="0 0 0" />
+      <origin xyz="0 0 0.149" rpy="0 0 0" />
       <parent link="${prefix}_laser_mount" />
       <child link="${prefix}_laser" />

File: jackal_description/urdf/accessories/sick_lms1xx_mount.urdf.xacro (robot description, xacro)
@@ -27,12 +27,6 @@
 <robot xmlns:xacro="http://www.ros.org/wiki/xacro">
   <xacro:include filename="$(find lms1xx)/urdf/sick_lms1xx.urdf.xacro" />
-  <xacro:macro name="sick_lms1xx_mount" params="prefix topic parent_link">
-    <xacro:sick_lms1xx frame="${prefix}_laser" topic="${topic}" />
-    <joint name="${prefix}_laser_mount_joint" type="fixed">
-      <origin xyz="$(optenv JACKAL_LASER_OFFSET 0 0 0)"
-              rpy="$(optenv JACKAL_LASER_RPY 0 0 0)" />
-      <parent link="${parent_link}" />
-      <child link="${prefix}_laser_mount" />
-    </joint>
+  <xacro:macro name="sick_lms1xx_mount" params="prefix topic">
+    <sick_lms1xx frame="${prefix}_laser" topic="${topic}" />
     <link name="${prefix}_laser_mount">
       <visual>

File: jackal_description/urdf/jackal.urdf.xacro (robot description, xacro)
@@ -80,4 +80,10 @@
     <origin xyz="${-wheelbase/2} ${-track/2} ${wheel_vertical_offset}" rpy="0 0 0" />
   </xacro:wheel>
+  <link name="base"></link>
+  <joint name="base_joint" type="fixed">
+    <origin xyz="0 0 0" rpy="0 0 0" />
+    <parent link="base"/>
+    <child link="base_link" />
+  </joint>
   <link name="base_link"></link>
   <joint name="base_link_joint" type="fixed">
